Commit message: first commit,uncomplete controller

File: ur_description/urdf/dual_ur5e.urdf.xacro (robot description, xacro)
@@ -38,18 +38,48 @@
     <origin xyz="0 -0.35 1.6" rpy="${PI/4*3} 0 0" />
   </joint>
-  <!-- robotieq 3f gripper -->
-  <xacro:include filename="$(find robotiq_3f_gripper_visualization)/cfg/robotiq-3f-gripper_articulated_macro.xacro" />
-  <!-- left gripper -->
-  <xacro:robotiq-3f-gripper_articulated prefix="left_"/>
-  <!-- right gripper -->
-  <xacro:robotiq-3f-gripper_articulated prefix="right_"/>
+  <!-- Simple box gripper for left arm -->
+  <link name="left_gripper">
+    <visual>
+      <origin xyz="0.05 0 0" rpy="0 ${PI/4*3} -${PI/2}"/>
+      <geometry>
+        <box size="0.1 0.1 0.1"/>
+      </geometry>
+      <material name="Blue">
+        <color rgba="0 0 1 1"/>
+      </material>
+    </visual>
+    <collision>
+      <origin xyz="0.05 0 0" rpy="0 ${PI/4*3} -${PI/2}"/>
+      <geometry>
+        <box size="0.1 0.1 0.1"/>
+      </geometry>
+    </collision>
+  </link>
+  <!-- Simple box gripper for right arm -->
+  <link name="right_gripper">
+    <visual>
+      <origin xyz="0.05 0 0" rpy="0 ${PI/4*3} -${PI/2}"/>
+      <geometry>
+        <box size="0.1 0.1 0.1"/>
+      </geometry>
+      <material name="Red">
+        <color rgba="1 0 0 1"/>
+      </material>
+    </visual>
+    <collision>
+      <origin xyz="0.05 0 0" rpy="0 ${PI/4*3} -${PI/2}"/>
+      <geometry>
+        <box size="0.1 0.1 0.1"/>
+      </geometry>
+    </collision>
+  </link>
   <joint name="left_gripper_joint" type="fixed">
     <parent link="left_ee_link" />
-    <child link = "left_palm" />
+    <child link = "left_gripper" />
     <origin xyz="0.05 0 0" rpy="0 ${PI/4*3} -${PI/2}" />
   </joint>
   <joint name="right_gripper_joint" type="fixed">
     <parent link="right_ee_link" />
-    <child link = "right_palm" />
+    <child link = "right_gripper" />
     <origin xyz="0.05 0 0" rpy="0 ${PI/4*3} -${PI/2}" />
   </joint>
