Commit message: add moveit

File: dual_ur_inspire_description/urdf/ur5e_moveit.urdf.xacro (robot description, xacro)
@@ -332,9 +332,9 @@
     <!-- <xacro:ur_arm_transmission prefix="${prefix}" /> -->
     <!-- <xacro:ur_arm_gazebo prefix="${prefix}" /> -->
-    <xacro:if value="$(arg use_gazebo)">
+    <!-- <xacro:if value="$(use_gazebo)"> -->
     <!-- Import Gazebo Classic definitions + plugin -->
       <xacro:include filename="$(find dual_ur_inspire_description)/urdf/ur_control.gazebo.xacro" />
       <xacro:ur_arm_gazebo prefix="${prefix}"/>
-    </xacro:if>
+    <!-- </xacro:if> -->
     <!-- ROS base_link to UR 'Base' Coordinates transform -->
     <link name="${prefix}base"/>

File: dual_ur_inspire_moveit_config/config/dual_ur_inspire.urdf.xacro (robot description, xacro)
@@ -37,15 +37,14 @@
 <!-- (1) UR5 -->
   <!-- <xacro:include filename="$(find dual_ur_inspire_description)/urdf/common.gazebo.xacro" /> -->
-  <xacro:include filename="$(find dual_ur_inspire_description)/urdf/ur5e_control.urdf.xacro" />
+  <xacro:include filename="$(find dual_ur_inspire_description)/urdf/ur5e_moveit.urdf.xacro" />
   <xacro:include filename="$(find dual_ur_inspire_description)/urdf/ur5e_control.ros2_control.xacro" />
   <!-- left arm -->
   <!-- <xacro:ur5e_robot prefix="left_" joint_limited="$(arg limited)" transmission_hw_interface="$(arg transmission_hw_interface)"/> -->
-  <xacro:ur5e_robot prefix="left_" joint_limited="$(arg limited)" use_gazebo="$(arg use_gazebo)"/>
-  <xacro:ur_arm_ros2_control prefix="left_" use_gazebo="$(arg use_gazebo)"/>
+  <xacro:ur5e_robot prefix="left_" joint_limited="false" use_gazebo="true"/>
+  <xacro:ur_arm_ros2_control prefix="left_" use_gazebo="true"/>
   <!-- right arm -->
   <!-- <xacro:ur5e_robot prefix="right_" joint_limited="$(arg limited)" transmission_hw_interface="$(arg transmission_hw_interface)"/> -->
-  <xacro:ur5e_robot prefix="right_" joint_limited="$(arg limited)" use_gazebo="$(arg use_gazebo)"/>
-  <xacro:ur_arm_ros2_control prefix="right_" use_gazebo="$(arg use_gazebo)"/>
-  <xacro:if value="$(arg use_gazebo)">
+  <xacro:ur5e_robot prefix="right_" joint_limited="false" use_gazebo="true"/>
+  <xacro:ur_arm_ros2_control prefix="right_" use_gazebo="true"/>
     <!-- Gazebo Plugin Loader -->
     <gazebo>
@@ -54,5 +53,4 @@
       </plugin>
     </gazebo>
-  </xacro:if>
   <joint name="left_arm_joint" type="fixed">
     <parent link="stand" />
@@ -68,11 +66,12 @@
   <xacro:include filename="$(find dual_ur_inspire_description)/urdf/inspire_hand_left.xacro" />
   <xacro:include filename="$(find dual_ur_inspire_description)/urdf/inspire_hand_right.xacro" />
+  <xacro:property name="use_sim_time" value="true" />
   <!-- Instantiate left Inspire hand -->
-  <xacro:inspire_hand_left prefix="left_hand_" parent_link="left_ee_link">
+  <!-- <xacro:inspire_hand_left prefix="left_hand_" parent_link="left_ee_link">
     <origin xyz="0 0 0" rpy="0 0 ${PI/2}" />
-  </xacro:inspire_hand_left>
+  </xacro:inspire_hand_left> -->
   <!-- Instantiate right Inspire hand -->
-  <xacro:inspire_hand_right prefix="right_hand_" parent_link="right_ee_link">
+  <!-- <xacro:inspire_hand_right prefix="right_hand_" parent_link="right_ee_link">
     <origin xyz="0 0 0" rpy="0 0 ${PI/2}" />
-  </xacro:inspire_hand_right>
+  </xacro:inspire_hand_right> -->
 </robot>
