Commit message: realize mimic by controller

File: dual_ur_inspire_description/urdf/inspire_hand_left.ros2_control.xacro (robot description, xacro)
@@ -28,6 +28,30 @@
         <state_interface name="velocity"/>
       </joint>
+      <joint name="${prefix}L_thumb_intermediate_joint">
+        <command_interface name="position">
+          <param name="min">0.0</param>
+          <param name="max">0.8</param>
+        </command_interface>
+        <state_interface name="position"/>
+        <state_interface name="velocity"/>
+      </joint>
+      <joint name="${prefix}L_thumb_distal_joint">
+        <command_interface name="position">
+          <param name="min">0.0</param>
+          <param name="max">0.8</param>
+        </command_interface>
+        <state_interface name="position"/>
+        <state_interface name="velocity"/>
+      </joint>
       <!-- Index finger joint -->
       <joint name="${prefix}L_index_proximal_joint">
+        <command_interface name="position">
+          <param name="min">0.0</param>
+          <param name="max">1.7</param>
+        </command_interface>
+        <state_interface name="position"/>
+        <state_interface name="velocity"/>
+      </joint>
+      <joint name="${prefix}L_index_intermediate_joint">
         <command_interface name="position">
           <param name="min">0.0</param>
@@ -46,6 +70,22 @@
         <state_interface name="velocity"/>
       </joint>
+      <joint name="${prefix}L_middle_intermediate_joint">
+        <command_interface name="position">
+          <param name="min">0.0</param>
+          <param name="max">1.7</param>
+        </command_interface>
+        <state_interface name="position"/>
+        <state_interface name="velocity"/>
+      </joint>
       <!-- Ring finger joint -->
       <joint name="${prefix}L_ring_proximal_joint">
+        <command_interface name="position">
+          <param name="min">0.0</param>
+          <param name="max">1.7</param>
+        </command_interface>
+        <state_interface name="position"/>
+        <state_interface name="velocity"/>
+      </joint>
+      <joint name="${prefix}L_ring_intermediate_joint">
         <command_interface name="position">
           <param name="min">0.0</param>
@@ -64,4 +104,12 @@
         <state_interface name="velocity"/>
       </joint>
+      <joint name="${prefix}L_pinky_intermediate_joint">
+        <command_interface name="position">
+          <param name="min">0.0</param>
+          <param name="max">1.7</param>
+        </command_interface>
+        <state_interface name="position"/>
+        <state_interface name="velocity"/>
+      </joint>
     </ros2_control>
   </xacro:macro>

File: dual_ur_inspire_description/urdf/inspire_hand_left.xacro (robot description, xacro)
@@ -194,8 +194,8 @@
         effort="1"
         velocity="0.5" />
-      <mimic
+      <!-- <mimic
         joint="${prefix}L_thumb_proximal_pitch_joint"
         multiplier="1.6"
-        offset="0" />
+        offset="0" /> -->
     </joint>
     <link name="${prefix}L_thumb_distal">
@@ -246,11 +246,11 @@
       <limit
         lower="0"
-        upper="0.8"
-        effort="1"
-        velocity="0.5" />
-      <mimic
+        upper="1.2"
+        effort="1"
+        velocity="0.5" />
+      <!-- <mimic
         joint="${prefix}L_thumb_proximal_pitch_joint"
-        multiplier="1.6"
-        offset="0" />
+        multiplier="2.4"
+        offset="0" /> -->
     </joint>
     <link name="${prefix}L_thumb_tip">
@@ -374,8 +374,8 @@
         effort="1"
         velocity="0.5" />
-      <mimic
+      <!-- <mimic
         joint="${prefix}L_index_proximal_joint"
         multiplier="1"
-        offset="0" />
+        offset="0" /> -->
     </joint>
     <link name="${prefix}L_index_tip">
@@ -499,8 +499,8 @@
         effort="1"
         velocity="0.5" />
-      <mimic
+      <!-- <mimic
         joint="${prefix}L_middle_proximal_joint"
         multiplier="1"
-        offset="0" />
+        offset="0" /> -->
     </joint>
     <link name="${prefix}L_middle_tip">
@@ -624,8 +624,8 @@
         effort="1"
         velocity="0.5" />
-      <mimic
+      <!-- <mimic
         joint="${prefix}L_ring_proximal_joint"
         multiplier="1"
-        offset="0" />
+        offset="0" /> -->
     </joint>
     <link name="${prefix}L_ring_tip">
@@ -749,8 +749,8 @@
         effort="1"
         velocity="0.5" />
-      <mimic
+      <!-- <mimic
         joint="${prefix}L_pinky_proximal_joint"
         multiplier="1"
-        offset="0" />
+        offset="0" /> -->
     </joint>
     <link name="${prefix}L_pinky_tip">

File: dual_ur_inspire_description/urdf/inspire_hand_right.ros2_control.xacro (robot description, xacro)
@@ -28,6 +28,30 @@
         <state_interface name="velocity"/>
       </joint>
+      <joint name="${prefix}R_thumb_intermediate_joint">
+        <command_interface name="position">
+          <param name="min">0.0</param>
+          <param name="max">0.8</param>
+        </command_interface>
+        <state_interface name="position"/>
+        <state_interface name="velocity"/>
+      </joint>
+      <joint name="${prefix}R_thumb_distal_joint">
+        <command_interface name="position">
+          <param name="min">0.0</param>
+          <param name="max">0.8</param>
+        </command_interface>
+        <state_interface name="position"/>
+        <state_interface name="velocity"/>
+      </joint>
       <!-- Index finger joint -->
       <joint name="${prefix}R_index_proximal_joint">
+        <command_interface name="position">
+          <param name="min">0.0</param>
+          <param name="max">1.7</param>
+        </command_interface>
+        <state_interface name="position"/>
+        <state_interface name="velocity"/>
+      </joint>
+      <joint name="${prefix}R_index_intermediate_joint">
         <command_interface name="position">
           <param name="min">0.0</param>
@@ -46,6 +70,22 @@
         <state_interface name="velocity"/>
       </joint>
+      <joint name="${prefix}R_middle_intermediate_joint">
+        <command_interface name="position">
+          <param name="min">0.0</param>
+          <param name="max">1.7</param>
+        </command_interface>
+        <state_interface name="position"/>
+        <state_interface name="velocity"/>
+      </joint>
       <!-- Ring finger joint -->
       <joint name="${prefix}R_ring_proximal_joint">
+        <command_interface name="position">
+          <param name="min">0.0</param>
+          <param name="max">1.7</param>
+        </command_interface>
+        <state_interface name="position"/>
+        <state_interface name="velocity"/>
+      </joint>
+      <joint name="${prefix}R_ring_intermediate_joint">
         <command_interface name="position">
           <param name="min">0.0</param>
@@ -64,4 +104,12 @@
         <state_interface name="velocity"/>
       </joint>
+      <joint name="${prefix}R_pinky_intermediate_joint">
+        <command_interface name="position">
+          <param name="min">0.0</param>
+          <param name="max">1.7</param>
+        </command_interface>
+        <state_interface name="position"/>
+        <state_interface name="velocity"/>
+      </joint>
     </ros2_control>
   </xacro:macro>

File: dual_ur_inspire_description/urdf/inspire_hand_right.xacro (robot description, xacro)
@@ -196,8 +196,8 @@
         effort="1"
         velocity="0.5" />
-      <mimic
+      <!-- <mimic
         joint="${prefix}R_thumb_proximal_pitch_joint"
         multiplier="1.6"
-        offset="0" />
+        offset="0" /> -->
     </joint>
     <link name="${prefix}R_thumb_distal">
@@ -251,8 +251,8 @@
         effort="1"
         velocity="0.5" />
-      <mimic
+      <!-- <mimic
         joint="${prefix}R_thumb_proximal_pitch_joint"
         multiplier="2.4"
-        offset="0" />
+        offset="0" /> -->
     </joint>
     <link name="${prefix}R_thumb_tip">
@@ -376,8 +376,8 @@
         effort="1"
         velocity="0.5" />
-      <mimic
+      <!-- <mimic
         joint="${prefix}R_index_proximal_joint"
         multiplier="1"
-        offset="0" />
+        offset="0" /> -->
     </joint>
     <link name="${prefix}R_index_tip">
@@ -501,8 +501,8 @@
         effort="1"
         velocity="0.5" />
-      <mimic
+      <!-- <mimic
         joint="${prefix}R_middle_proximal_joint"
         multiplier="1"
-        offset="0" />
+        offset="0" /> -->
     </joint>
     <link name="${prefix}R_middle_tip">
@@ -626,8 +626,8 @@
         effort="1"
         velocity="0.5" />
-      <mimic
+      <!-- <mimic
         joint="${prefix}R_ring_proximal_joint"
         multiplier="1"
-        offset="0" />
+        offset="0" /> -->
     </joint>
     <link name="${prefix}R_ring_tip">
@@ -751,8 +751,8 @@
         effort="1"
         velocity="0.5" />
-      <mimic
+      <!-- <mimic
         joint="${prefix}R_pinky_proximal_joint"
         multiplier="1"
-        offset="0" />
+        offset="0" /> -->
     </joint>
     <link name="${prefix}R_pinky_tip">
