Commit message: add ros2_control

File: dual_ur_inspire_description/urdf/dual_ur_inspire_control.urdf.xacro (robot description, xacro)
@@ -36,15 +36,23 @@
   </joint>
 <!-- (1) UR5 -->
-  <xacro:include filename="$(find dual_ur_inspire_description)/urdf/common.gazebo.xacro" />
+  <!-- <xacro:include filename="$(find dual_ur_inspire_description)/urdf/common.gazebo.xacro" /> -->
   <xacro:include filename="$(find dual_ur_inspire_description)/urdf/ur5e_control.urdf.xacro" />
   <xacro:include filename="$(find dual_ur_inspire_description)/urdf/ur5e_control.ros2_control.xacro" />
   <!-- left arm -->
   <!-- <xacro:ur5e_robot prefix="left_" joint_limited="$(arg limited)" transmission_hw_interface="$(arg transmission_hw_interface)"/> -->
-  <xacro:ur5e_robot prefix="left_" joint_limited="$(arg limited)"/>
-  <xacro:ur_arm_ros2_control prefix="left_" />
+  <xacro:ur5e_robot prefix="left_" joint_limited="$(arg limited)" use_gazebo="$(arg use_gazebo)"/>
+  <xacro:ur_arm_ros2_control prefix="left_" use_gazebo="$(arg use_gazebo)"/>
   <!-- right arm -->
   <!-- <xacro:ur5e_robot prefix="right_" joint_limited="$(arg limited)" transmission_hw_interface="$(arg transmission_hw_interface)"/> -->
-  <xacro:ur5e_robot prefix="right_" joint_limited="$(arg limited)"/>
-  <xacro:ur_arm_ros2_control prefix="right_" />
+  <xacro:ur5e_robot prefix="right_" joint_limited="$(arg limited)" use_gazebo="$(arg use_gazebo)"/>
+  <xacro:ur_arm_ros2_control prefix="right_" use_gazebo="$(arg use_gazebo)"/>
+  <xacro:if value="$(arg use_gazebo)">
+    <!-- Gazebo Plugin Loader -->
+    <gazebo>
+      <plugin filename="gz_ros2_control-system" name="gz_ros2_control::GazeboSimROS2ControlPlugin">
+        <parameters>$(find dual_ur_inspire_description)/config/dual_arm_inspire_controller.yaml</parameters>
+      </plugin>
+    </gazebo>
+  </xacro:if>
   <joint name="left_arm_joint" type="fixed">
     <parent link="stand" />

File: dual_ur_inspire_description/urdf/ur5e_control.ros2_control.xacro (robot description, xacro)
@@ -1,9 +1,13 @@
 <?xml version="1.0"?>
 <robot xmlns:xacro="http://ros.org/wiki/xacro">
-  <xacro:macro name="ur_arm_ros2_control" params="prefix">
+  <xacro:macro name="ur_arm_ros2_control" params="prefix use_gazebo:=^|true">
     <ros2_control name="${prefix}ur_arm_system" type="system">
       <hardware>
-        <!-- <plugin>ros2_control_demo_hardware/RRBotSystemPositionOnlyHardware</plugin> -->
-        <plugin>gazebo_ros2_control/GazeboSystem</plugin>
+        <xacro:if value="${use_gazebo}">
+          <plugin>gz_ros2_control/GazeboSimSystem</plugin>
+        </xacro:if>
+        <xacro:unless value="${use_gazebo}">
+          <plugin>gz_ros2_control/IsaacsimHardWare</plugin>
+        </xacro:unless>
       </hardware>
       <!-- Each joint definition -->

File: dual_ur_inspire_description/urdf/ur5e_control.urdf.xacro (robot description, xacro)
@@ -2,5 +2,5 @@
 <robot xmlns:xacro="http://ros.org/wiki/xacro">
   <!-- <xacro:include filename="$(find dual_ur_inspire_description)/urdf/ur.transmission.xacro" /> -->
-  <xacro:include filename="$(find dual_ur_inspire_description)/urdf/ur_control.gazebo.xacro" />
+  <!-- <xacro:include filename="$(find dual_ur_inspire_description)/urdf/ur_control.gazebo.xacro" /> -->
   <xacro:macro name="cylinder_inertial" params="radius length mass *origin">
     <inertial>
@@ -12,5 +12,5 @@
     </inertial>
   </xacro:macro>
-  <xacro:macro name="ur5e_robot" params="prefix joint_limited
+  <xacro:macro name="ur5e_robot" params="prefix joint_limited use_gazebo
     shoulder_pan_lower_limit:=${-pi}    shoulder_pan_upper_limit:=${pi}
     shoulder_lift_lower_limit:=${-pi}    shoulder_lift_upper_limit:=${pi}
@@ -330,5 +330,10 @@
     </link>
     <!-- <xacro:ur_arm_transmission prefix="${prefix}" /> -->
-    <xacro:ur_arm_gazebo prefix="${prefix}" />
+    <!-- <xacro:ur_arm_gazebo prefix="${prefix}" /> -->
+    <xacro:if value="$(arg use_gazebo)">
+    <!-- Import Gazebo Classic definitions + plugin -->
+      <xacro:include filename="$(find dual_ur_inspire_description)/urdf/ur_control.gazebo.xacro" />
+      <xacro:ur_arm_gazebo prefix="${prefix}"/>
+    </xacro:if>
     <!-- ROS base_link to UR 'Base' Coordinates transform -->
     <link name="${prefix}base"/>

File: dual_ur_inspire_description/urdf/ur_control.gazebo.xacro (robot description, xacro)
@@ -2,9 +2,9 @@
   <xacro:macro name="ur_arm_gazebo" params="prefix">
     <!-- Gazebo Plugin Loader -->
-    <gazebo>
-      <plugin name="gazebo_ros2_control" filename="libgazebo_ros2_control.so">
-        <ros2_control_name>${prefix}ur_arm_gazebo</ros2_control_name>
+    <!-- <gazebo>
+      <plugin filename="gz_ros2_control-system" name="gz_ros2_control::GazeboSimROS2ControlPlugin">
+        <parameters>$(find dual_ur_inspire_description)/config/dual_arm_inspire_controller.yaml</parameters>
       </plugin>
-    </gazebo>
+    </gazebo> -->
     <!-- Link Self-Collision Settings -->
     <gazebo reference="${prefix}shoulder_link">

Commit message: add joint cmd param

File: dual_ur_inspire_description/urdf/dual_ur_inspire_control.urdf.xacro (robot description, xacro)
@@ -42,9 +42,9 @@
   <!-- <xacro:ur5e_robot prefix="left_" joint_limited="$(arg limited)" transmission_hw_interface="$(arg transmission_hw_interface)"/> -->
   <xacro:ur5e_robot prefix="left_" joint_limited="$(arg limited)" use_gazebo="$(arg use_gazebo)"/>
-  <xacro:ur_arm_ros2_control prefix="left_" use_gazebo="$(arg use_gazebo)"/>
+  <xacro:ur_arm_ros2_control prefix="left_" command_topic="left_arm_cmd" use_gazebo="$(arg use_gazebo)"/>
   <!-- right arm -->
   <!-- <xacro:ur5e_robot prefix="right_" joint_limited="$(arg limited)" transmission_hw_interface="$(arg transmission_hw_interface)"/> -->
   <xacro:ur5e_robot prefix="right_" joint_limited="$(arg limited)" use_gazebo="$(arg use_gazebo)"/>
-  <xacro:ur_arm_ros2_control prefix="right_" use_gazebo="$(arg use_gazebo)"/>
+  <xacro:ur_arm_ros2_control prefix="right_" command_topic="right_arm_cmd" use_gazebo="$(arg use_gazebo)"/>
   <xacro:if value="$(arg use_gazebo)">
     <!-- Gazebo Plugin Loader -->

File: dual_ur_inspire_description/urdf/ur5e_control.ros2_control.xacro (robot description, xacro)
@@ -1,5 +1,6 @@
 <?xml version="1.0"?>
 <robot xmlns:xacro="http://ros.org/wiki/xacro">
-  <xacro:macro name="ur_arm_ros2_control" params="prefix use_gazebo:=^|true">
+  <xacro:macro name="ur_arm_ros2_control" params="prefix command_topic use_gazebo:=^|true">
+    <xacro:property name="joint_cmd_topic" value="/${command_topic}" />
     <ros2_control name="${prefix}ur_arm_system" type="system">
       <hardware>
@@ -9,5 +10,5 @@
         <xacro:unless value="${use_gazebo}">
           <plugin>topic_based_ros2_control/TopicBasedSystem</plugin>
-          <param name="joint_commands_topic">/joint_command</param>
+          <param name="joint_commands_topic">${joint_cmd_topic}</param>
           <param name="joint_states_topic">/joint_states</param>
         </xacro:unless>

File: dual_ur_inspire_moveit_config/config/dual_ur_inspire_moveit.urdf.xacro (robot description, xacro)
@@ -42,15 +42,15 @@
   <!-- <xacro:ur5e_robot prefix="left_" joint_limited="$(arg limited)" transmission_hw_interface="$(arg transmission_hw_interface)"/> -->
   <xacro:ur5e_robot prefix="left_" joint_limited="false" use_gazebo="true"/>
-  <xacro:ur_arm_ros2_control prefix="left_" use_gazebo="true"/>
+  <xacro:ur_arm_ros2_control prefix="left_" command_topic="left_arm_cmd" use_gazebo="true"/>
   <!-- right arm -->
   <!-- <xacro:ur5e_robot prefix="right_" joint_limited="$(arg limited)" transmission_hw_interface="$(arg transmission_hw_interface)"/> -->
   <xacro:ur5e_robot prefix="right_" joint_limited="false" use_gazebo="true"/>
-  <xacro:ur_arm_ros2_control prefix="right_" use_gazebo="true"/>
+  <xacro:ur_arm_ros2_control prefix="right_" command_topic="right_arm_cmd" use_gazebo="true"/>
     <!-- Gazebo Plugin Loader -->
-    <gazebo>
+    <!-- <gazebo>
       <plugin filename="gz_ros2_control-system" name="gz_ros2_control::GazeboSimROS2ControlPlugin">
         <parameters>$(find dual_ur_inspire_description)/config/dual_arm_inspire_controller.yaml</parameters>
       </plugin>
-    </gazebo>
+    </gazebo> -->
   <joint name="left_arm_joint" type="fixed">
     <parent link="stand" />

Commit message: add reserve shoulder lift joint

File: dual_ur_inspire_description/urdf/dual_ur_inspire_control.urdf.xacro (robot description, xacro)
@@ -41,9 +41,9 @@
   <!-- left arm -->
   <!-- <xacro:ur5e_robot prefix="left_" joint_limited="$(arg limited)" transmission_hw_interface="$(arg transmission_hw_interface)"/> -->
-  <xacro:ur5e_robot prefix="left_" joint_limited="$(arg limited)" use_gazebo="$(arg use_gazebo)"/>
+  <xacro:ur5e_robot prefix="left_" joint_limited="$(arg limited)" use_gazebo="$(arg use_gazebo)" reverse_shoulder_lift="false"/>
   <xacro:ur_arm_ros2_control prefix="left_" command_topic="left_arm_cmd" use_gazebo="$(arg use_gazebo)"/>
   <!-- right arm -->
   <!-- <xacro:ur5e_robot prefix="right_" joint_limited="$(arg limited)" transmission_hw_interface="$(arg transmission_hw_interface)"/> -->
-  <xacro:ur5e_robot prefix="right_" joint_limited="$(arg limited)" use_gazebo="$(arg use_gazebo)"/>
+  <xacro:ur5e_robot prefix="right_" joint_limited="$(arg limited)" use_gazebo="$(arg use_gazebo)" reverse_shoulder_lift="true"/>
   <xacro:ur_arm_ros2_control prefix="right_" command_topic="right_arm_cmd" use_gazebo="$(arg use_gazebo)"/>
   <xacro:if value="$(arg use_gazebo)">

File: dual_ur_inspire_description/urdf/ur5e_control.urdf.xacro (robot description, xacro)
@@ -12,5 +12,5 @@
     </inertial>
   </xacro:macro>
-  <xacro:macro name="ur5e_robot" params="prefix joint_limited use_gazebo
+  <xacro:macro name="ur5e_robot" params="prefix joint_limited use_gazebo reverse_shoulder_lift
     shoulder_pan_lower_limit:=${-pi}    shoulder_pan_upper_limit:=${pi}
     shoulder_lift_lower_limit:=${-pi}    shoulder_lift_upper_limit:=${pi}
@@ -135,5 +135,10 @@
       <parent link="${prefix}shoulder_link" />
       <child link = "${prefix}upper_arm_link" />
-      <origin xyz="0.0 ${shoulder_offset} 0.0" rpy="0.0 ${pi / 2.0} 0.0" />
+      <xacro:if value="${reverse_shoulder_lift}">
+        <origin xyz="0.0 ${shoulder_offset} 0.0" rpy="0.0 ${pi / 2.0} ${pi}" />
+      </xacro:if>
+      <xacro:unless value="${reverse_shoulder_lift}">
+        <origin xyz="0.0 ${shoulder_offset} 0.0" rpy="0.0 ${pi / 2.0} 0.0" />
+      </xacro:unless>
       <axis xyz="0 1 0" />
       <xacro:unless value="${joint_limited}">

File: dual_ur_inspire_description/urdf/ur5e_moveit.urdf.xacro (robot description, xacro)
@@ -12,5 +12,5 @@
     </inertial>
   </xacro:macro>
-  <xacro:macro name="ur5e_robot" params="prefix joint_limited use_gazebo
+  <xacro:macro name="ur5e_robot" params="prefix joint_limited use_gazebo reverse_shoulder_lift
     shoulder_pan_lower_limit:=${-pi}    shoulder_pan_upper_limit:=${pi}
     shoulder_lift_lower_limit:=${-pi}    shoulder_lift_upper_limit:=${pi}
@@ -135,5 +135,10 @@
       <parent link="${prefix}shoulder_link" />
       <child link = "${prefix}upper_arm_link" />
-      <origin xyz="0.0 ${shoulder_offset} 0.0" rpy="0.0 ${pi / 2.0} 0.0" />
+      <xacro:if value="${reverse_shoulder_lift}">
+        <origin xyz="0.0 ${shoulder_offset} 0.0" rpy="0.0 ${pi / 2.0} ${pi}" />
+      </xacro:if>
+      <xacro:unless value="${reverse_shoulder_lift}">
+        <origin xyz="0.0 ${shoulder_offset} 0.0" rpy="0.0 ${pi / 2.0} 0.0" />
+      </xacro:unless>
       <axis xyz="0 1 0" />
       <xacro:unless value="${joint_limited}">

File: dual_ur_inspire_moveit_config/config/dual_ur_inspire_moveit.urdf.xacro (robot description, xacro)
@@ -41,9 +41,9 @@
   <!-- left arm -->
   <!-- <xacro:ur5e_robot prefix="left_" joint_limited="$(arg limited)" transmission_hw_interface="$(arg transmission_hw_interface)"/> -->
-  <xacro:ur5e_robot prefix="left_" joint_limited="false" use_gazebo="true"/>
+  <xacro:ur5e_robot prefix="left_" joint_limited="false" use_gazebo="true" reverse_shoulder_lift="false"/>
   <xacro:ur_arm_ros2_control prefix="left_" command_topic="left_arm_cmd" use_gazebo="true"/>
   <!-- right arm -->
   <!-- <xacro:ur5e_robot prefix="right_" joint_limited="$(arg limited)" transmission_hw_interface="$(arg transmission_hw_interface)"/> -->
-  <xacro:ur5e_robot prefix="right_" joint_limited="false" use_gazebo="true"/>
+  <xacro:ur5e_robot prefix="right_" joint_limited="false" use_gazebo="true" reverse_shoulder_lift="true"/>
   <xacro:ur_arm_ros2_control prefix="right_" command_topic="right_arm_cmd" use_gazebo="true"/>
     <!-- Gazebo Plugin Loader -->

Commit message: completed reserve shoulder,add joint state filter

File: dual_ur_inspire_description/urdf/dual_ur_inspire_control.urdf.xacro (robot description, xacro)
@@ -41,9 +41,9 @@
   <!-- left arm -->
   <!-- <xacro:ur5e_robot prefix="left_" joint_limited="$(arg limited)" transmission_hw_interface="$(arg transmission_hw_interface)"/> -->
-  <xacro:ur5e_robot prefix="left_" joint_limited="$(arg limited)" use_gazebo="$(arg use_gazebo)" reverse_shoulder_lift="false"/>
+  <xacro:ur5e_robot prefix="left_" joint_limited="$(arg limited)" use_gazebo="$(arg use_gazebo)" reverse_arm="false"/>
   <xacro:ur_arm_ros2_control prefix="left_" command_topic="left_arm_cmd" use_gazebo="$(arg use_gazebo)"/>
   <!-- right arm -->
   <!-- <xacro:ur5e_robot prefix="right_" joint_limited="$(arg limited)" transmission_hw_interface="$(arg transmission_hw_interface)"/> -->
-  <xacro:ur5e_robot prefix="right_" joint_limited="$(arg limited)" use_gazebo="$(arg use_gazebo)" reverse_shoulder_lift="true"/>
+  <xacro:ur5e_robot prefix="right_" joint_limited="$(arg limited)" use_gazebo="$(arg use_gazebo)" reverse_arm="true"/>
   <xacro:ur_arm_ros2_control prefix="right_" command_topic="right_arm_cmd" use_gazebo="$(arg use_gazebo)"/>
   <xacro:if value="$(arg use_gazebo)">

File: dual_ur_inspire_description/urdf/inspire_hand_left.xacro (robot description, xacro)
@@ -194,8 +194,8 @@
         effort="1"
         velocity="0.5" />
-      <!-- <mimic
+      <mimic
         joint="${prefix}L_thumb_proximal_pitch_joint"
         multiplier="1.6"
-        offset="0" /> -->
+        offset="0" />
     </joint>
     <link name="${prefix}L_thumb_distal">
@@ -249,8 +249,8 @@
         effort="1"
         velocity="0.5" />
-      <!-- <mimic
+      <mimic
         joint="${prefix}L_thumb_proximal_pitch_joint"
         multiplier="2.4"
-        offset="0" /> -->
+        offset="0" />
     </joint>
     <link name="${prefix}L_thumb_tip">
@@ -374,8 +374,8 @@
         effort="1"
         velocity="0.5" />
-      <!-- <mimic
+      <mimic
         joint="${prefix}L_index_proximal_joint"
         multiplier="1"
-        offset="0" /> -->
+        offset="0" />
     </joint>
     <link name="${prefix}L_index_tip">
@@ -499,8 +499,8 @@
         effort="1"
         velocity="0.5" />
-      <!-- <mimic
+      <mimic
         joint="${prefix}L_middle_proximal_joint"
         multiplier="1"
-        offset="0" /> -->
+        offset="0" />
     </joint>
     <link name="${prefix}L_middle_tip">
@@ -624,8 +624,8 @@
         effort="1"
         velocity="0.5" />
-      <!-- <mimic
+      <mimic
         joint="${prefix}L_ring_proximal_joint"
         multiplier="1"
-        offset="0" /> -->
+        offset="0" />
     </joint>
     <link name="${prefix}L_ring_tip">
@@ -749,8 +749,8 @@
         effort="1"
         velocity="0.5" />
-      <!-- <mimic
+      <mimic
         joint="${prefix}L_pinky_proximal_joint"
         multiplier="1"
-        offset="0" /> -->
+        offset="0" />
     </joint>
     <link name="${prefix}L_pinky_tip">

File: dual_ur_inspire_description/urdf/inspire_hand_right.xacro (robot description, xacro)
@@ -196,8 +196,8 @@
         effort="1"
         velocity="0.5" />
-      <!-- <mimic
+      <mimic
         joint="${prefix}R_thumb_proximal_pitch_joint"
         multiplier="1.6"
-        offset="0" /> -->
+        offset="0" />
     </joint>
     <link name="${prefix}R_thumb_distal">
@@ -251,8 +251,8 @@
         effort="1"
         velocity="0.5" />
-      <!-- <mimic
+      <mimic
         joint="${prefix}R_thumb_proximal_pitch_joint"
         multiplier="2.4"
-        offset="0" /> -->
+        offset="0" />
     </joint>
     <link name="${prefix}R_thumb_tip">
@@ -376,8 +376,8 @@
         effort="1"
         velocity="0.5" />
-      <!-- <mimic
+      <mimic
         joint="${prefix}R_index_proximal_joint"
         multiplier="1"
-        offset="0" /> -->
+        offset="0" />
     </joint>
     <link name="${prefix}R_index_tip">
@@ -501,8 +501,8 @@
         effort="1"
         velocity="0.5" />
-      <!-- <mimic
+      <mimic
         joint="${prefix}R_middle_proximal_joint"
         multiplier="1"
-        offset="0" /> -->
+        offset="0" />
     </joint>
     <link name="${prefix}R_middle_tip">
@@ -626,8 +626,8 @@
         effort="1"
         velocity="0.5" />
-      <!-- <mimic
+      <mimic
         joint="${prefix}R_ring_proximal_joint"
         multiplier="1"
-        offset="0" /> -->
+        offset="0" />
     </joint>
     <link name="${prefix}R_ring_tip">
@@ -751,8 +751,8 @@
         effort="1"
         velocity="0.5" />
-      <!-- <mimic
+      <mimic
         joint="${prefix}R_pinky_proximal_joint"
         multiplier="1"
-        offset="0" /> -->
+        offset="0" />
     </joint>
     <link name="${prefix}R_pinky_tip">

File: dual_ur_inspire_description/urdf/ur5e_control.urdf.xacro (robot description, xacro)
@@ -12,5 +12,5 @@
     </inertial>
   </xacro:macro>
-  <xacro:macro name="ur5e_robot" params="prefix joint_limited use_gazebo reverse_shoulder_lift
+  <xacro:macro name="ur5e_robot" params="prefix joint_limited use_gazebo reverse_arm
     shoulder_pan_lower_limit:=${-pi}    shoulder_pan_upper_limit:=${pi}
     shoulder_lift_lower_limit:=${-pi}    shoulder_lift_upper_limit:=${pi}
@@ -135,8 +135,8 @@
       <parent link="${prefix}shoulder_link" />
       <child link = "${prefix}upper_arm_link" />
-      <xacro:if value="${reverse_shoulder_lift}">
-        <origin xyz="0.0 ${shoulder_offset} 0.0" rpy="0.0 ${pi / 2.0} ${pi}" />
-      </xacro:if>
-      <xacro:unless value="${reverse_shoulder_lift}">
+      <xacro:if value="${reverse_arm}">
+        <origin xyz="0.0 ${shoulder_offset} 0.0" rpy="${pi} ${pi / 2.0 + pi} ${pi}" />
+      </xacro:if>
+      <xacro:unless value="${reverse_arm}">
         <origin xyz="0.0 ${shoulder_offset} 0.0" rpy="0.0 ${pi / 2.0} 0.0" />
       </xacro:unless>
@@ -214,5 +214,10 @@
       <parent link="${prefix}forearm_link" />
       <child link = "${prefix}wrist_1_link" />
-      <origin xyz="0.0 0.0 ${forearm_length}" rpy="0.0 ${pi / 2.0} 0.0" />
+      <xacro:if value="${reverse_arm}">
+        <origin xyz="0.0 0.0 ${forearm_length}" rpy="${pi} ${pi / 2.0 + pi} ${pi}" />
+      </xacro:if>
+      <xacro:unless value="${reverse_arm}">
+        <origin xyz="0.0 0.0 ${forearm_length}" rpy="0.0 ${pi / 2.0} 0.0" />
+      </xacro:unless>
       <axis xyz="0 1 0" />
       <xacro:unless value="${joint_limited}">

File: dual_ur_inspire_description/urdf/ur5e_moveit.urdf.xacro (robot description, xacro)
@@ -12,5 +12,5 @@
     </inertial>
   </xacro:macro>
-  <xacro:macro name="ur5e_robot" params="prefix joint_limited use_gazebo reverse_shoulder_lift
+  <xacro:macro name="ur5e_robot" params="prefix joint_limited use_gazebo reverse_arm
     shoulder_pan_lower_limit:=${-pi}    shoulder_pan_upper_limit:=${pi}
     shoulder_lift_lower_limit:=${-pi}    shoulder_lift_upper_limit:=${pi}
@@ -135,8 +135,8 @@
       <parent link="${prefix}shoulder_link" />
       <child link = "${prefix}upper_arm_link" />
-      <xacro:if value="${reverse_shoulder_lift}">
-        <origin xyz="0.0 ${shoulder_offset} 0.0" rpy="0.0 ${pi / 2.0} ${pi}" />
-      </xacro:if>
-      <xacro:unless value="${reverse_shoulder_lift}">
+      <xacro:if value="${reverse_arm}">
+        <origin xyz="0.0 ${shoulder_offset} 0.0" rpy="${pi} ${pi / 2.0 + pi} ${pi}" />
+      </xacro:if>
+      <xacro:unless value="${reverse_arm}">
         <origin xyz="0.0 ${shoulder_offset} 0.0" rpy="0.0 ${pi / 2.0} 0.0" />
       </xacro:unless>
@@ -214,5 +214,10 @@
       <parent link="${prefix}forearm_link" />
       <child link = "${prefix}wrist_1_link" />
-      <origin xyz="0.0 0.0 ${forearm_length}" rpy="0.0 ${pi / 2.0} 0.0" />
+      <xacro:if value="${reverse_arm}">
+        <origin xyz="0.0 0.0 ${forearm_length}" rpy="${pi} ${pi / 2.0 + pi} ${pi}" />
+      </xacro:if>
+      <xacro:unless value="${reverse_arm}">
+        <origin xyz="0.0 0.0 ${forearm_length}" rpy="0.0 ${pi / 2.0} 0.0" />
+      </xacro:unless>
       <axis xyz="0 1 0" />
       <xacro:unless value="${joint_limited}">

File: dual_ur_inspire_moveit_config/config/dual_ur_inspire_moveit.urdf.xacro (robot description, xacro)
@@ -41,9 +41,9 @@
   <!-- left arm -->
   <!-- <xacro:ur5e_robot prefix="left_" joint_limited="$(arg limited)" transmission_hw_interface="$(arg transmission_hw_interface)"/> -->
-  <xacro:ur5e_robot prefix="left_" joint_limited="false" use_gazebo="true" reverse_shoulder_lift="false"/>
+  <xacro:ur5e_robot prefix="left_" joint_limited="false" use_gazebo="true" reverse_arm="false"/>
   <xacro:ur_arm_ros2_control prefix="left_" command_topic="left_arm_cmd" use_gazebo="true"/>
   <!-- right arm -->
   <!-- <xacro:ur5e_robot prefix="right_" joint_limited="$(arg limited)" transmission_hw_interface="$(arg transmission_hw_interface)"/> -->
-  <xacro:ur5e_robot prefix="right_" joint_limited="false" use_gazebo="true" reverse_shoulder_lift="true"/>
+  <xacro:ur5e_robot prefix="right_" joint_limited="false" use_gazebo="true" reverse_arm="true"/>
   <xacro:ur_arm_ros2_control prefix="right_" command_topic="right_arm_cmd" use_gazebo="true"/>
     <!-- Gazebo Plugin Loader -->
