Commit message: add moveit interface

File: dual_ur_inspire_description/urdf/dual_ur_inspire_control.urdf.xacro (robot description, xacro)
@@ -41,9 +41,9 @@
   <!-- left arm -->
   <!-- <xacro:ur5e_robot prefix="left_" joint_limited="$(arg limited)" transmission_hw_interface="$(arg transmission_hw_interface)"/> -->
-  <xacro:ur5e_robot prefix="left_" joint_limited="$(arg limited)" use_gazebo="$(arg use_gazebo)" reverse_arm="false"/>
+  <xacro:ur5e_robot prefix="left_" joint_limited="$(arg limited)" use_gazebo="$(arg use_gazebo)" reverse_arm="true"/>
   <xacro:ur_arm_ros2_control prefix="left_" command_topic="left_arm_cmd" use_gazebo="$(arg use_gazebo)"/>
   <!-- right arm -->
   <!-- <xacro:ur5e_robot prefix="right_" joint_limited="$(arg limited)" transmission_hw_interface="$(arg transmission_hw_interface)"/> -->
-  <xacro:ur5e_robot prefix="right_" joint_limited="$(arg limited)" use_gazebo="$(arg use_gazebo)" reverse_arm="true"/>
+  <xacro:ur5e_robot prefix="right_" joint_limited="$(arg limited)" use_gazebo="$(arg use_gazebo)" reverse_arm="false"/>
   <xacro:ur_arm_ros2_control prefix="right_" command_topic="right_arm_cmd" use_gazebo="$(arg use_gazebo)"/>
   <xacro:if value="$(arg use_gazebo)">
@@ -73,10 +73,10 @@
   <!-- <xacro:inspire_hand_left prefix="left_hand_" parent_link="left_ee_link">
     <origin xyz="0 0 0" rpy="0 0 ${PI/2}" />
-  </xacro:inspire_hand_left>
-  <xacro:inspire_hand_left_ros2_control prefix="left_hand_" use_gazebo="$(arg use_gazebo)"/> -->
+  </xacro:inspire_hand_left> -->
+  <!-- <xacro:inspire_hand_left_ros2_control prefix="left_hand_" use_gazebo="$(arg use_gazebo)"/> -->
   <!-- Instantiate right Inspire hand -->
   <!-- <xacro:inspire_hand_right prefix="right_hand_" parent_link="right_ee_link">
     <origin xyz="0 0 0" rpy="0 0 ${PI/2}" />
-  </xacro:inspire_hand_right>
-  <xacro:inspire_hand_right_ros2_control prefix="right_hand_" use_gazebo="$(arg use_gazebo)"/> -->
+  </xacro:inspire_hand_right> -->
+  <!-- <xacro:inspire_hand_right_ros2_control prefix="right_hand_" use_gazebo="$(arg use_gazebo)"/> -->
 </robot>

File: dual_ur_inspire_description/urdf/ur5e_control.urdf.xacro (robot description, xacro)
@@ -293,5 +293,10 @@
       <parent link="${prefix}wrist_2_link" />
       <child link = "${prefix}wrist_3_link" />
-      <origin xyz="0.0 0.0 ${wrist_2_length}" rpy="0.0 0.0 0.0" />
+      <xacro:if value="${reverse_arm}">
+        <origin xyz="0.0 0.0 ${wrist_2_length}" rpy="0.0 ${pi} 0.0" />
+      </xacro:if>
+      <xacro:unless value="${reverse_arm}">
+        <origin xyz="0.0 0.0 ${wrist_2_length}" rpy="0.0 0.0 0.0" />
+      </xacro:unless>
       <axis xyz="0 1 0" />
       <xacro:unless value="${joint_limited}">

File: dual_ur_inspire_description/urdf/ur5e_moveit.urdf.xacro (robot description, xacro)
@@ -293,5 +293,10 @@
       <parent link="${prefix}wrist_2_link" />
       <child link = "${prefix}wrist_3_link" />
-      <origin xyz="0.0 0.0 ${wrist_2_length}" rpy="0.0 0.0 0.0" />
+      <xacro:if value="${reverse_arm}">
+        <origin xyz="0.0 0.0 ${wrist_2_length}" rpy="0.0 ${pi} 0.0" />
+      </xacro:if>
+      <xacro:unless value="${reverse_arm}">
+        <origin xyz="0.0 0.0 ${wrist_2_length}" rpy="0.0 0.0 0.0" />
+      </xacro:unless>
       <axis xyz="0 1 0" />
       <xacro:unless value="${joint_limited}">

File: dual_ur_inspire_moveit_config/config/dual_ur_inspire_moveit.urdf (robot description, URDF)
Before this commit: robot dual_ur_robotiq, 58 links, 57 joints
Joints:
- joint left_shoulder_lift_joint: origin xyz=0.0 0.138 0.0 rpy=0.0 1.5707963267948966 0.0 -> xyz=0.0 0.138 0.0 rpy=3.141592653589793 4.71238898038469 3.141592653589793
- joint left_wrist_1_joint: origin xyz=0.0 0.0 0.392 rpy=0.0 1.5707963267948966 0.0 -> xyz=0.0 0.0 0.392 rpy=3.141592653589793 4.71238898038469 3.141592653589793
- joint left_wrist_3_joint: origin xyz=0.0 0.0 0.1 rpy=0.0 0.0 0.0 -> xyz=0.0 0.0 0.1 rpy=0.0 3.141592653589793 0.0
- joint right_shoulder_lift_joint: origin xyz=0.0 0.138 0.0 rpy=3.141592653589793 4.71238898038469 3.141592653589793 -> xyz=0.0 0.138 0.0 rpy=0.0 1.5707963267948966 0.0
- joint right_wrist_1_joint: origin xyz=0.0 0.0 0.392 rpy=3.141592653589793 4.71238898038469 3.141592653589793 -> xyz=0.0 0.0 0.392 rpy=0.0 1.5707963267948966 0.0

File: dual_ur_inspire_moveit_config/config/dual_ur_inspire_moveit.urdf.xacro (robot description, xacro)
@@ -41,9 +41,9 @@
   <!-- left arm -->
   <!-- <xacro:ur5e_robot prefix="left_" joint_limited="$(arg limited)" transmission_hw_interface="$(arg transmission_hw_interface)"/> -->
-  <xacro:ur5e_robot prefix="left_" joint_limited="false" use_gazebo="true" reverse_arm="false"/>
+  <xacro:ur5e_robot prefix="left_" joint_limited="false" use_gazebo="true" reverse_arm="true"/>
   <xacro:ur_arm_ros2_control prefix="left_" command_topic="left_arm_cmd" use_gazebo="true"/>
   <!-- right arm -->
   <!-- <xacro:ur5e_robot prefix="right_" joint_limited="$(arg limited)" transmission_hw_interface="$(arg transmission_hw_interface)"/> -->
-  <xacro:ur5e_robot prefix="right_" joint_limited="false" use_gazebo="true" reverse_arm="true"/>
+  <xacro:ur5e_robot prefix="right_" joint_limited="false" use_gazebo="true" reverse_arm="false"/>
   <xacro:ur_arm_ros2_control prefix="right_" command_topic="right_arm_cmd" use_gazebo="true"/>
     <!-- Gazebo Plugin Loader -->
@@ -68,16 +68,13 @@
   <xacro:include filename="$(find dual_ur_inspire_description)/urdf/inspire_hand_right.xacro" />
   <xacro:include filename="$(find dual_ur_inspire_description)/urdf/inspire_hand_right.ros2_control.xacro" /> -->
-  <!-- <xacro:include filename="$(find dual_ur_inspire_description)/urdf/inspire_hand_gazebo.xacro" /> -->
   <!-- Instantiate left Inspire hand -->
   <!-- <xacro:inspire_hand_left prefix="left_hand_" parent_link="left_ee_link">
     <origin xyz="0 0 0" rpy="0 0 ${PI/2}" />
-  </xacro:inspire_hand_left>
-  <xacro:inspire_hand_left_ros2_control prefix="left_hand_" use_gazebo="true"/> -->
-  <!-- <xacro:inspire_hand_gazebo prefix="left_hand_L"/> -->
+  </xacro:inspire_hand_left> -->
+  <!-- <xacro:inspire_hand_left_ros2_control prefix="left_hand_" use_gazebo="true"/> -->
   <!-- Instantiate right Inspire hand -->
   <!-- <xacro:inspire_hand_right prefix="right_hand_" parent_link="right_ee_link">
     <origin xyz="0 0 0" rpy="0 0 ${PI/2}" />
-  </xacro:inspire_hand_right>
-  <xacro:inspire_hand_right_ros2_control prefix="right_hand_" use_gazebo="true"/> -->
-  <!-- <xacro:inspire_hand_gazebo prefix="left_hand_R"/> -->
+  </xacro:inspire_hand_right> -->
+  <!-- <xacro:inspire_hand_right_ros2_control prefix="right_hand_" use_gazebo="true"/> -->
 </robot>
