Commit message: add ur driver hardwareinterface

File: dual_arm_model/urdf/ur5e.urdf.xacro (robot description, xacro)
@@ -139,5 +139,5 @@
       <child link = "${prefix}upper_arm_link" />
       <xacro:if value="${reverse_arm}">
-        <origin xyz="0.0 ${shoulder_offset} 0.0" rpy="${pi} ${pi / 2.0 + pi} ${pi}" />
+        <origin xyz="0.0 ${shoulder_offset} 0.0" rpy="${pi} ${pi / 2.0} ${pi}" />
       </xacro:if>
       <xacro:unless value="${reverse_arm}">
@@ -218,5 +218,5 @@
       <child link = "${prefix}wrist_1_link" />
       <xacro:if value="${reverse_arm}">
-        <origin xyz="0.0 0.0 ${forearm_length}" rpy="${pi} ${pi / 2.0 + pi} ${pi}" />
+        <origin xyz="0.0 0.0 ${forearm_length}" rpy="${pi} ${pi / 2.0} ${pi}" />
       </xacro:if>
       <xacro:unless value="${reverse_arm}">
@@ -260,8 +260,8 @@
       <child link = "${prefix}wrist_2_link" />
       <xacro:if value="${reverse_arm}">
-        <origin xyz="0.0 ${wrist_1_length} 0.0" rpy="0.0 0.0 ${-PI/2}" />
-      </xacro:if>
-      <xacro:unless value="${reverse_arm}">
-        <origin xyz="0.0 ${wrist_1_length} 0.0" rpy="0.0 0.0 ${PI/2}" />
+        <origin xyz="0.0 ${wrist_1_length} 0.0" rpy="0.0 0.0 0.0" />
+      </xacro:if>
+      <xacro:unless value="${reverse_arm}">
+        <origin xyz="0.0 ${wrist_1_length} 0.0" rpy="0.0 0.0 0.0" />
       </xacro:unless>
       <axis xyz="0 0 1" />
@@ -302,8 +302,8 @@
       <child link = "${prefix}wrist_3_link" />
       <xacro:if value="${reverse_arm}">
-        <origin xyz="0.0 0.0 ${wrist_2_length}" rpy="0.0 ${-pi/2} 0.0" />
-      </xacro:if>
-      <xacro:unless value="${reverse_arm}">
-        <origin xyz="0.0 0.0 ${wrist_2_length}" rpy="0.0 ${-pi/2} 0.0" />
+        <origin xyz="0.0 0.0 ${wrist_2_length}" rpy="0.0 0.0 0.0" />
+      </xacro:if>
+      <xacro:unless value="${reverse_arm}">
+        <origin xyz="0.0 0.0 ${wrist_2_length}" rpy="0.0 0.0 0.0" />
       </xacro:unless>
       <axis xyz="0 1 0" />
