Commit message: change to rtde

File: dual_arm_model/urdf/ur.ros2_control.xacro (robot description, xacro)
@@ -23,5 +23,5 @@
     <ros2_control name="${prefix}ur_arm_system" type="system">
       <hardware>
-          <plugin>ur_robot_driver/URPositionHardwareInterface</plugin>
+          <!-- <plugin>ur_robot_driver/URPositionHardwareInterface</plugin>
           <param name="robot_ip">${robot_ip}</param>
           <param name="script_filename">${script_filename}</param>
@@ -48,5 +48,15 @@
           <param name="tool_device_name">${tool_device_name}</param>
           <param name="tool_tcp_port">${tool_tcp_port}</param>
-          <param name="keep_alive_count">${keep_alive_count}</param>
+          <param name="keep_alive_count">${keep_alive_count}</param> -->
+          <plugin>mock_components/GenericSystem</plugin>
+          <param name="mock_sensor_commands">true</param>
+          <param name="state_following_offset">0.0</param>
+          <param name="calculate_dynamics">true</param>
+          <param name="joints">
+            [${prefix}shoulder_pan_joint, ${prefix}shoulder_lift_joint, ${prefix}elbow_joint,
+            ${prefix}wrist_1_joint, ${prefix}wrist_2_joint, ${prefix}wrist_3_joint]
+          </param>
+          <param name="command_interfaces">[position]</param>
+          <param name="state_interfaces">[position, velocity]</param>
       </hardware>
       <!-- Each joint definition -->

File: dual_ur_inspire_bringup/urdf/real_bot_arm.urdf (robot description, URDF)
Before this commit: robot dual_ur_robotiq, 22 links, 21 joints
Links:
- added link left_base_link_inertia, mass 4.0; collision mesh filename=package://ur_description/meshes/ur5/collision/base.stl; visual mesh filename=package://ur_description/meshes/ur5/visual/base.dae
- added link left_flange
- added link left_ft_frame
- added link right_base_link_inertia, mass 4.0; collision mesh filename=package://ur_description/meshes/ur5/collision/base.stl; visual mesh filename=package://ur_description/meshes/ur5/visual/base.dae
- added link right_flange
- added link right_ft_frame
- link left_base_link: mass 4.0 -> None; geometry 
- link left_forearm_link: mass 2.275 -> 2.33; geometry collision mesh filename=package://ur_description/meshes/ur5/collision/forearm.stl; visual mesh filename=package://ur_description/meshes/ur5/visual/forearm.dae
- link left_shoulder_link: geometry collision mesh filename=package://ur_description/meshes/ur5/collision/shoulder.stl; visual mesh filename=package://ur_description/meshes/ur5/visual/shoulder.dae
- link left_upper_arm_link: geometry collision mesh filename=package://ur_description/meshes/ur5/collision/upperarm.stl; visual mesh filename=package://ur_description/meshes/ur5/visual/upperarm.dae
- link left_wrist_1_link: geometry collision mesh filename=package://ur_description/meshes/ur5/collision/wrist1.stl; visual mesh filename=package://ur_description/meshes/ur5/visual/wrist1.dae
- link left_wrist_2_link: geometry collision mesh filename=package://ur_description/meshes/ur5/collision/wrist2.stl; visual mesh filename=package://ur_description/meshes/ur5/visual/wrist2.dae
- link left_wrist_3_link: geometry collision mesh filename=package://ur_description/meshes/ur5/collision/wrist3.stl; visual mesh filename=package://ur_description/meshes/ur5/visual/wrist3.dae
- link right_base_link: mass 4.0 -> None; geometry 
- link right_forearm_link: mass 2.275 -> 2.33; geometry collision mesh filename=package://ur_description/meshes/ur5/collision/forearm.stl; visual mesh filename=package://ur_description/meshes/ur5/visual/forearm.dae
- link right_shoulder_link: geometry collision mesh filename=package://ur_description/meshes/ur5/collision/shoulder.stl; visual mesh filename=package://ur_description/meshes/ur5/visual/shoulder.dae
- link right_upper_arm_link: geometry collision mesh filename=package://ur_description/meshes/ur5/collision/upperarm.stl; visual mesh filename=package://ur_description/meshes/ur5/visual/upperarm.dae
- link right_wrist_1_link: geometry collision mesh filename=package://ur_description/meshes/ur5/collision/wrist1.stl; visual mesh filename=package://ur_description/meshes/ur5/visual/wrist1.dae
- link right_wrist_2_link: geometry collision mesh filename=package://ur_description/meshes/ur5/collision/wrist2.stl; visual mesh filename=package://ur_description/meshes/ur5/visual/wrist2.dae
- link right_wrist_3_link: geometry collision mesh filename=package://ur_description/meshes/ur5/collision/wrist3.stl; visual mesh filename=package://ur_description/meshes/ur5/visual/wrist3.dae
Joints:
- removed joint left_wrist_3_link-tool0_fixed_joint
- removed joint right_wrist_3_link-tool0_fixed_joint
- added joint left_base_link-base_link_inertia: type fixed, parent left_base_link, child left_base_link_inertia, origin xyz=0 0 0 rpy=0 0 3.141592653589793
- added joint left_flange-tool0: type fixed, parent left_flange, child left_tool0, origin xyz=0 0 0 rpy=1.5707963267948966 0 1.5707963267948966
- added joint left_wrist_3-flange: type fixed, parent left_wrist_3_link, child left_flange, origin xyz=0 0 0 rpy=0 -1.5707963267948966 -1.5707963267948966
- added joint left_wrist_3_link-ft_frame: type fixed, parent left_wrist_3_link, child left_ft_frame, origin xyz=0 0 0 rpy=3.141592653589793 0 0
- added joint right_base_link-base_link_inertia: type fixed, parent right_base_link, child right_base_link_inertia, origin xyz=0 0 0 rpy=0 0 3.141592653589793
- added joint right_flange-tool0: type fixed, parent right_flange, child right_tool0, origin xyz=0 0 0 rpy=1.5707963267948966 0 1.5707963267948966
- added joint right_wrist_3-flange: type fixed, parent right_wrist_3_link, child right_flange, origin xyz=0 0 0 rpy=0 -1.5707963267948966 -1.5707963267948966
- added joint right_wrist_3_link-ft_frame: type fixed, parent right_wrist_3_link, child right_ft_frame, origin xyz=0 0 0 rpy=3.141592653589793 0 0
- joint left_base_link-base_fixed_joint: origin xyz=0 0 0 rpy=0 0 -3.141592653589793 -> xyz=0 0 0 rpy=0 0 3.141592653589793
- joint left_ee_fixed_joint: origin xyz=0.0 0.1 0.0 rpy=0.0 0.0 1.5707963267948966 -> xyz=0.0 0.0 0.0 rpy=0.0 -1.5707963267948966 1.5707963267948966
- joint left_elbow_joint: axis 0 1 0 -> 0 0 1; limit lower=-3.141592653589793 upper=3.141592653589793 effort=150.0 velocity=3.14 -> lower=-3.141592653589793 upper=3.141592653589793 effort=150.0 velocity=6.283185307179586; origin xyz=0.0 -0.131 0.425 rpy=0.0 0.0 0.0 -> xyz=-0.425 0 0 rpy=0 0 0
- joint left_shoulder_lift_joint: axis 0 1 0 -> 0 0 1; limit lower=-3.141592653589793 upper=3.141592653589793 effort=150.0 velocity=3.14 -> lower=-6.283185307179586 upper=6.283185307179586 effort=150.0 velocity=6.283185307179586; origin xyz=0.0 0.138 0.0 rpy=0.0 1.5707963267948966 0.0 -> xyz=0 0 0 rpy=1.570796327 0 0
- joint left_shoulder_pan_joint: limit lower=-3.141592653589793 upper=3.141592653589793 effort=150.0 velocity=3.14 -> lower=-6.283185307179586 upper=6.283185307179586 effort=150.0 velocity=6.283185307179586; origin xyz=0.0 0.0 0.163 rpy=0.0 0.0 0.0 -> xyz=0 0 0.089159 rpy=0 0 0; parent left_base_link -> left_base_link_inertia
- joint left_wrist_1_joint: axis 0 1 0 -> 0 0 1; limit lower=-3.141592653589793 upper=3.141592653589793 effort=28.0 velocity=6.28 -> lower=-6.283185307179586 upper=6.283185307179586 effort=28.0 velocity=6.283185307179586; origin xyz=0.0 0.0 0.392 rpy=0.0 1.5707963267948966 0.0 -> xyz=-0.39225 0 0.10915 rpy=0 0 0
- joint left_wrist_2_joint: limit lower=-3.141592653589793 upper=3.141592653589793 effort=28.0 velocity=6.28 -> lower=-6.283185307179586 upper=6.283185307179586 effort=28.0 velocity=6.283185307179586; origin xyz=0.0 0.127 0.0 rpy=0.0 0.0 0.0 -> xyz=0 -0.09465 -1.941303950897609e-11 rpy=1.570796327 0 0
- joint left_wrist_3_joint: axis 0 1 0 -> 0 0 1; limit lower=-3.141592653589793 upper=3.141592653589793 effort=28.0 velocity=6.28 -> lower=-6.283185307179586 upper=6.283185307179586 effort=28.0 velocity=6.283185307179586; origin xyz=0.0 0.0 0.1 rpy=0.0 0.0 0.0 -> xyz=0 0.0823 -1.688001216681175e-11 rpy=1.570796326589793 3.141592653589793 3.141592653589793
- joint right_arm_joint: origin xyz=0 -0.25 1.05 rpy=1.5707963267948966 0 0 -> xyz=0 -0.25 1.05 rpy=1.5707963267948966 3.141592653589793 0
- joint right_base_link-base_fixed_joint: origin xyz=0 0 0 rpy=0 0 -3.141592653589793 -> xyz=0 0 0 rpy=0 0 3.141592653589793
- joint right_ee_fixed_joint: origin xyz=0.0 0.1 0.0 rpy=0.0 0.0 1.5707963267948966 -> xyz=0.0 0.0 0.0 rpy=0.0 -1.5707963267948966 1.5707963267948966
- joint right_elbow_joint: axis 0 1 0 -> 0 0 1; limit lower=-3.141592653589793 upper=3.141592653589793 effort=150.0 velocity=3.14 -> lower=-3.141592653589793 upper=3.141592653589793 effort=150.0 velocity=6.283185307179586; origin xyz=0.0 -0.131 0.425 rpy=0.0 0.0 0.0 -> xyz=-0.425 0 0 rpy=0 0 0
- joint right_shoulder_lift_joint: axis 0 1 0 -> 0 0 1; limit lower=-3.141592653589793 upper=3.141592653589793 effort=150.0 velocity=3.14 -> lower=-6.283185307179586 upper=6.283185307179586 effort=150.0 velocity=6.283185307179586; origin xyz=0.0 0.138 0.0 rpy=3.141592653589793 1.5707963267948966 3.141592653589793 -> xyz=0 0 0 rpy=1.570796327 0 0
- joint right_shoulder_pan_joint: limit lower=-3.141592653589793 upper=3.141592653589793 effort=150.0 velocity=3.14 -> lower=-6.283185307179586 upper=6.283185307179586 effort=150.0 velocity=6.283185307179586; origin xyz=0.0 0.0 0.163 rpy=0.0 0.0 3.141592653589793 -> xyz=0 0 0.089159 rpy=0 0 0; parent right_base_link -> right_base_link_inertia
- joint right_wrist_1_joint: axis 0 1 0 -> 0 0 1; limit lower=-3.141592653589793 upper=3.141592653589793 effort=28.0 velocity=6.28 -> lower=-6.283185307179586 upper=6.283185307179586 effort=28.0 velocity=6.283185307179586; origin xyz=0.0 0.0 0.392 rpy=3.141592653589793 1.5707963267948966 3.141592653589793 -> xyz=-0.39225 0 0.10915 rpy=0 0 0
- joint right_wrist_2_joint: limit lower=-3.141592653589793 upper=3.141592653589793 effort=28.0 velocity=6.28 -> lower=-6.283185307179586 upper=6.283185307179586 effort=28.0 velocity=6.283185307179586; origin xyz=0.0 0.127 0.0 rpy=0.0 0.0 0.0 -> xyz=0 -0.09465 -1.941303950897609e-11 rpy=1.570796327 0 0
- joint right_wrist_3_joint: axis 0 1 0 -> 0 0 1; limit lower=-3.141592653589793 upper=3.141592653589793 effort=28.0 velocity=6.28 -> lower=-6.283185307179586 upper=6.283185307179586 effort=28.0 velocity=6.283185307179586; origin xyz=0.0 0.0 0.1 rpy=0.0 0.0 0.0 -> xyz=0 0.0823 -1.688001216681175e-11 rpy=1.570796326589793 3.141592653589793 3.141592653589793
